File: Bus_switch.kicad_sch (KiCad schematic)
At the start: 15 parts, among them J3 Conn_01x04_Pin, U1 SN74CB3Q3384APW

Commit message: done
Parts:
- removed R11, R2, R3, R5, R7, R8, R9: 10kΩ, PCM_JLCPCB:R_0402, symbol PCM_JLCPCB-Resistors:0402,10kΩ
Other:
- company: (none) -> MiniModucard System
- title: MMS3 Hat template small (Change Me) -> MMS3 Hat Relay
