File: Hardware/CH32V003.kicad_sch (KiCad schematic)
At the start: 11 parts, among them J4 WCH Link, J5 Program, U3 CH32V003FxPx, X1 X322525MOB4SI

Commit message: Ver 1.2 - Fixed SDA SCL mixup
Changed lines of the file:
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@@
 		(title "MMS3 Hat Relay")
 		(date "2026-06-08")
-		(rev "1.1")
+		(rev "1.2")
 		(company "MiniModucard System")
 		(comment 1 "Wojciech Szafrański")
@@
 	)
 	(label "PC2"
-		(at 46.99 97.79 0)
+		(at 46.99 93.98 0)
 		(effects
 			(font
@@
 	)
 	(label "PC1"
-		(at 46.99 93.98 0)
-		(effects
-			(font
+		(at 46.99 97.79 0)
+		(effects
+			(font
